File: src/0x0A/0x0A.sch (KiCad schematic (older format))
At the start: 5 parts

Commit message: new file:   imgs/better.png 	modified:   src/0x0A/0x0A-cache.lib 	modified:   src/0x0A/0x0A.sch 	modified:   src/0x0A/antenna.sch 	modified:   src/0x0A/audio.sch 	modified:   src/0x0A/buttons.sch 	new file:   src/0x0A/cameras.sch 	modified:   src/0x0A/display.sch 	modified:   src/0x0A/gpio.sch 	modified:   src/0x0A/pwr.sch 	modified:   src/0x0A/sensors.sch 	modified:   src/0x0A/sim.sch 	modified:   src/0x0A/uart.sch 	modified:   src/0x0A/usb.sch 	new file:   src/models/body.obj 	new file:   src/models/phone.FCStd 	new file:   src/models/screen.obj
Added 3D models, integrated front & rear cameras, flash light, reformatting & more
Parts:
- removed U? (x5): SC600Y, XCVR_SC600Y, symbol SC600Y:SC600Y
- added D?: LED, symbol Device:LED
- added R?: 0R, symbol Device:R_Small_US
- added U? (x5): SC600YNAPAE53UGADA, SnapEDA Library:XCVR_SC600YNAPAE53UGADA, symbol SC600YNAPAE53UGADA:SC600YNAPAE53UGADA
Connections:
- net 1.2V_DVDD_FRONT: now also U?.15 (LDO23_1P2)
- net 1.2V_DVDD_REAR: now also U?.13 (LDO2_1P1)
- net 1.8V_GPIO: now also U?.9 (LDO5_1P8)
- net 1.8V_LCD: now also U?.10 (LDO6_1P8)
- net 2.85V_LCD: now also U?.12 (LDO17_2P85)
- net 2.8V_AVDD: now also U?.14 (LDO22_2P8)
- net 2.8V_SENSE: now also U?.11 (LDO10_2P8)
- net ANT_DRX: now also U?.149 (ANT_DRX)
- net ANT_GNSS: now also U?.134 (ANT_GNSS)
- net ANT_MAIN: now also U?.19 (ANT_MAIN)
- net ANT_WIFI: now also U?.129 (ANT_WIFI/BT)
- net BAT_MINUS: now also U?.28 (BAT_MINUS)
- net BAT_PLUS: now also U?.27 (BAT_PLUS)
- net BAT_THERM: now also U?.29 (BAT_THERM)
- net DSI0_CLKN: now also U?.116 (DSI0_CLK_N)
- net DSI0_CLKP: now also U?.115 (DSI0_CLK_P)
- net DSI0_D0N: now also U?.118 (DSI0_LN0_N)
- net DSI0_D0P: now also U?.117 (DSI0_LN0_P)
- net DSI0_D1N: now also U?.120 (DSI0_LN1_N)
- net DSI0_D1P: now also U?.119 (DSI0_LN1_P)
- net DSI0_D2N: now also U?.122 (DSI0_LN2_N)
- net DSI0_D2P: now also U?.121 (DSI0_LN2_P)
- net DSI0_D3N: now also U?.124 (DSI0_LN3_N)
- net DSI0_D3P: now also U?.123 (DSI0_LN3_P)
- net DSI1_CLKN: now also U?.103 (DSI1_CLK_N)
- net DSI1_CLKP: now also U?.102 (DSI1_CLK_P)
- net DSI1_D0N: now also U?.105 (DSI1_LN0_N)
- net DSI1_D0P: now also U?.104 (DSI1_LN0_P)
- net DSI1_D1N: now also U?.107 (DSI1_LN1_N)
- net DSI1_D1P: now also U?.106 (DSI1_LN1_P)
- net DSI1_D2N: now also U?.109 (DSI1_LN2_N)
- net DSI1_D2P: now also U?.108 (DSI1_LN2_P)
- net DSI1_D3N: now also U?.111 (DSI1_LN3_N)
- net DSI1_D3P: now also U?.110 (DSI1_LN3_P)
- net GND: now also R?.2, U?.101 (GND), U?.112 (GND), U?.125 (GND), U?.128 (GND), U?.130 (GND), U?.133 (GND), U?.135 (GND), U?.148 (GND), U?.150 (GND), U?.154 (GND), U?.155 (GND), U?.156 (GND), U?.157 (GND), U?.158 (GND), U?.159 (GND), U?.163 (GND), U?.164 (GND), U?.165 (GND), U?.166 (GND), U?.170 (GND), U?.173 (GND), U?.176 (GND), U?.18 (GND), U?.182 (GND), U?.193 (GND), U?.195 (GND), U?.20 (GND), U?.212 (GND), U?.213 (GND), U?.214 (GND), U?.218 (GND), U?.219 (GND), U?.222 (GND), U?.225 (GND), U?.235 (GND), U?.239 (GND), U?.240 (GND), U?.243 (GND), U?.245 (GND), U?.246 (GND), U?.247 (GND), U?.248 (GND), U?.249 (GND), U?.250 (GND), U?.251 (GND), U?.252 (GND), U?.253 (GND), U?.254 (GND), U?.255 (GND), U?.256 (GND), U?.257 (GND), U?.258 (GND), U?.259 (GND), U?.260 (GND), U?.261 (GND), U?.262 (GND), U?.263 (GND), U?.264 (GND), U?.265 (GND), U?.266 (GND), U?.267 (GND), U?.268 (GND), U?.269 (GND), U?.270 (GND), U?.271 (GND), U?.272 (GND), U?.273 (GND), U?.274 (GND), U?.275 (GND), U?.276 (GND), U?.277 (GND), U?.278 (GND), U?.279 (GND), U?.280 (GND), U?.281 (GND), U?.282 (GND), U?.283 (GND), U?.284 (GND), U?.285 (GND), U?.286 (GND), U?.287 (GND), U?.288 (GND), U?.289 (GND), U?.290 (GND), U?.291 (GND), U?.292 (GND), U?.293 (GND), U?.294 (GND), U?.295 (GND), U?.296 (GND), U?.297 (GND), U?.298 (GND), U?.299 (GND), U?.3 (GND), U?.300 (GND), U?.301 (GND), U?.302 (GND), U?.303 (GND), U?.304 (GND), U?.305 (GND), U?.306 (GND), U?.307 (GND), U?.308 (GND), U?.309 (GND), U?.31 (GND), U?.310 (GND), U?.311 (GND), U?.312 (GND), U?.313 (GND), U?.314 (GND), U?.315 (GND), U?.316 (GND), U?.317 (GND), U?.318 (GND), U?.319 (GND), U?.320 (GND), U?.321 (GND), U?.322 (GND), U?.323 (GND), U?.34 (GND), U?.35 (GND), U?.4 (GND), U?.40 (GND), U?.41 (GND), U?.42 (GND), U?.43 (GND), U?.47 (GND), U?.56 (GND), U?.62 (GND), U?.87 (GND), U?.98 (GND)
- net LCD0_ID: now also U?.153 (PMI_ADC)
- net LCD0_TE: now also U?.126 (LCD0_TE)
- net LCD1_ID: now also U?.151 (PMU_MPP2)
- net LCD1_RST: now also U?.113 (LCD1_RST)
- net LCD1_TE: now also U?.114 (LCD1_TE)
- net LCDO_RST: now also U?.127 (LCD0_RST)
- net LCD_BL_A: now also U?.21 (LCD_BL_A)
- net LCD_BL_K1: now also U?.22 (LCD_BL_K1)
- net LCD_BL_K2: now also U?.23 (LCD_BL_K2)
- net MIC1_N: now also U?.45 (MIC1_N)
- net MIC1_P: now also U?.44 (MIC1_P)
- net MIC2_P: now also U?.46 (MIC2_P)
- net MIC3_P: now also U?.169 (MIC3_P)
- net MIC_BIAS: now also U?.167 (MIC_BIAS)
- net PWR_KEY: now also U?.39 (SDC2_DATA0)
- net SIM_VDD: now also U?.141 (USIM1_VDD)
- net TP0_I2C_SCL: now also U?.140 (TP0_I2C_SCL)
- net TP0_I2C_SDA: now also U?.206 (TP0_I2C_SDA)
- net TP0_INT: now also U?.139 (TP0_INT)
- net TP0_RST: now also U?.138 (TP0_RST)
- net TP1_I2C_SCL: now also U?.205 (TP1_I2C_SCL)
- net TP1_I2C_SDA: now also U?.204 (TP1_SPI_SDA)
- net TP1_INT: now also U?.137 (TP1_INT)
- net TP1_RST: now also U?.136 (TP1_RST)
- net USB_BOOT: now also U?.57 (USB_BOOT)
- net USB_VBUS: now also U?.162 (USB_VBUS)
- net USIM1_CLK: now also U?.143 (USIM1_CLK)
- net USIM1_DATA: now also U?.142 (USIM1_DATA)
- net USIM1_DET: now also U?.145 (USIM1_DET)
- net USIM1_RST: now also U?.144 (USIM1_RST)
- net VBAT: now also U?.36 (VBAT), U?.37 (VBAT), U?.38 (VBAT)
- net VDD_RF: now also U?.1 (VDD_RF), U?.2 (VDD_RF)
- net VOL_DOWN: now also U?.147 (VOL_DOWN)
- net VOL_UP: now also U?.146 (VOL_UP)
- net VPH_PWR: now also U?.220 (VPH_PWR), U?.221 (VPH_PWR)
- net VRTC: now also U?.16 (VRTC)
- new net: D?.1 (K), R?.1
- new net CAM_I2C_SCL: U?.75 (CAN_I2C_SCL)
- new net CAM_I2C_SDA: U?.76 (CAM_I2C_SDA)
- new net FLASH_LED1: D?.2 (A), U?.26 (FLASH_LED1)
- new net FRONT_CLK_N: U?.78 (CSI2_CLK_N)
- new net FRONT_CLK_P: U?.77 (CSI2_CLK_P)
- new net FRONT_LN0_N: U?.80 (CSI2_LN0_N)
- new net FRONT_LN0_P: U?.79 (CSI2_LN0_P)
- new net FRONT_LN1_N: U?.82 (CSI2_LN1_N)
- new net FRONT_LN1_P: U?.81 (CSI2_LN1_P)
- new net FRONT_LN2_N: U?.84 (CSI2_LN2_N)
- new net FRONT_LN2_P: U?.83 (CSI2_LN2_P)
- new net FRONT_LN3_N: U?.86 (CSI2_LN3_N)
- new net FRONT_LN3_P: U?.85 (CSI2_LN3_P)
- new net FRONT_MCLK: U?.100 (SCAM_MCLK)
- new net FRONT_PWDN: U?.71 (SCAM_PWDN)
- new net FRONT_RESET: U?.72 (SCAM_RST)
- new net REAR_CLK_N: U?.89 (CSI0_CLK_N)
- new net REAR_CLK_P: U?.88 (CSI0_CLK_P)
- new net REAR_LN0_N: U?.91 (CSI0_LN0_N)
- new net REAR_LN0_P: U?.90 (CSI0_LN0_P)
- new net REAR_LN1_N: U?.93 (CSI0_LN1_N)
- new net REAR_LN1_P: U?.92 (CSI0_LN1_P)
- new net REAR_LN2_N: U?.95 (CSI0_LN2_N)
- new net REAR_LN2_P: U?.94 (CSI0_LN2_P)
- new net REAR_LN3_N: U?.97 (CSI0_LN3_N)
- new net REAR_LN3_P: U?.96 (CSI0_LN3_P)
- new net REAR_MCLK: U?.99 (MCAM_MCLK)
- new net REAR_PWDN: U?.73 (MCAM_PWDN)
- new net REAR_RESET: U?.74 (MCAM_RST)
- new net USB_CC1: U?.223 (USBC_CC1)
- new net USB_CC2: U?.224 (USBC_CC2)
- new net USB_D+: U?.32 (USB_DP)
- new net USB_D-: U?.33 (USB_DM)
- new net USB_SS_RX_M: U?.172 (USB_SS_RX_M)
- new net USB_SS_RX_P: U?.171 (USB_SS_RX_P)
- new net USB_SS_SEL: U?.226 (USB_SS_SEL)
- new net USB_SS_TX_M: U?.175 (USB_SS_TX_M)
- new net USB_SS_TX_P: U?.174 (USB_SS_TX_P)
- new net USIM2_CLK: U?.208 (USIM2_CLK)
- new net USIM2_RST: U?.207 (USIM2_RST)
- new net USIM_DATA: U?.209 (USIM_DATA)
- no-connect marks 13 -> 21
Other:
- note added: "Cameras"
- note added: "Flashlight"
- note added: "Might want to breakout\nthis camera just to allow\npeople to play around with\nhaving a depth cam"
- note added: "Not using active GPS"
- note added: "USB_OPT only needed for \nUSB micro, leave floating\nfor USB-C"

Commit message: Updated schematics, started working on board layout
Parts:
- R1: renamed from R?; footprint (none) -> Resistor_SMD:R_0402_1005Metric
- gave numbers to parts that had none: 2
Connections:
- net DCAM_CLK_P: now reaches U1.183 (CSI1_CLK_P)
- net DCAM_CLK_N: now reaches U1.184 (CSI1_CLK_N)
- net DCAM_LN0_P: now reaches U1.185 (CSI1_LN0_P)
- net DCAM_LN0_N: now reaches U1.186 (CSI1_LN0_N)
- net DCAM_LN1_P: now reaches U1.187 (CSI1_LN1_P)
- net DCAM_LN1_N: now reaches U1.188 (CSI1_LN1_N)
- net DCAM_LN2_P: now reaches U1.189 (CSI1_LN2_P)
- net DCAM_LN2_N: now reaches U1.190 (CSI1_LN2_N)
- net DCAM_LN3_P: now reaches U1.191 (CSI1_LN3_P)
- net DCAM_LN3_N: now reaches U1.192 (CSI1_LN3_N)
- net LDO12: now reaches U1.179 (SL_LDO12)
- net DCAM_RESET: now reaches U1.180 (DCAM_RST)
- net DCAM_PWDN: now reaches U1.181 (DCAM_PWN)
- net DCAM_MCLK: now reaches U1.194 (DCAM_MCLK)
- net EAR_N: now reaches U1.52 (EAR_N)
- net EAR_P: now reaches U1.53 (EAR_P)
- net SPK_N: now reaches U1.54 (SPK_N)
- net SPK_P: now reaches U1.55 (SPK_P)
- net SD_LD011: now reaches U1.63 (SD_LDO11)
- net SD_DET: now reaches U1.64 (SD_DET)
- net SD_DATA3: now reaches U1.65 (SD_DATA3)
- net SD_DATA2: now reaches U1.66 (SD_DATA2)
- net SD_DATA1: now reaches U1.67 (SD_DATA1)
- net SD_DATA0: now reaches U1.68 (SD_DATA0)
- net SD_CMD: now reaches U1.69 (SD_CMD)
- net SD_CLK: now reaches U1.70 (SD_CLK)
- net SENSE_SDA: now reaches U1.131 (SENSOR_I2C_SCL)
- net SENSE_SCL: now reaches U1.132 (SENSOR_I2C_SDA)
- net DCAM_I2C_SCL: now reaches U1.196 (DCAM_I2C_SCL)
- net DCAM_I2C_SDA: now reaches U1.197 (DCAM_I2C_SDA)
- net ALS_INT_N: now reaches U1.177 (GPIO_98)
- net GYRO_INT: now reaches U1.178 (GPIO_99)
- net FSYNC: now reaches U1.237 (GPIO_36)
- net MIC_GND: now reaches U1.168 (MIC_GND)
- net SIM2_VDD: now reaches U1.210 (USIM2_VDD)
- net MIC2_P: no longer names the net of U1.46 (MIC2_P)
- net USIM_DATA renamed USIM2_DATA
- no-connect marks 21 -> 34
Other:
- note added: "Headphone jack\n(Not implemented yet)"
- note removed: "Might want to breakout\nthis camera just to allow\npeople to play around with\nhaving a depth cam"
- moved on the sheet: D1, R1, U1A, U1E
