File: src/0x0A/antenna.sch (KiCad schematic (older format))
At the start: 17 parts

Commit message: new file:   imgs/better.png 	modified:   src/0x0A/0x0A-cache.lib 	modified:   src/0x0A/0x0A.sch 	modified:   src/0x0A/antenna.sch 	modified:   src/0x0A/audio.sch 	modified:   src/0x0A/buttons.sch 	new file:   src/0x0A/cameras.sch 	modified:   src/0x0A/display.sch 	modified:   src/0x0A/gpio.sch 	modified:   src/0x0A/pwr.sch 	modified:   src/0x0A/sensors.sch 	modified:   src/0x0A/sim.sch 	modified:   src/0x0A/uart.sch 	modified:   src/0x0A/usb.sch 	new file:   src/models/body.obj 	new file:   src/models/phone.FCStd 	new file:   src/models/screen.obj
Added 3D models, integrated front & rear cameras, flash light, reformatting & more
Parts:
- C28, C29, C30, C31, C32, C33, C34, C35, C36: renamed from C?; footprint (none) -> Capacitor_SMD:C_0603_1608Metric
- R11, R12, R13, R14: renamed from R?; footprint (none) -> Resistor_SMD:R_0402_1005Metric
- gave numbers to parts that had none: 4
Other:
- note added: "PI antenna circuits\nDon't place caps, leave for \nfuture tuning capabilities."
Changed lines of the file:
@@
 $Descr A4 11693 8268
 encoding utf-8
-Sheet 10 12
+Sheet 9 13
 Title "0x0A SmartPhone"
 Date "2022-09-01"
 Rev "1"
 Comp "HackThisPhone.com"
-Comment1 ""
+Comment1 "Designed By @NoahGWood for"
 Comment2 ""
 Comment3 ""
@@
 $EndDescr
 $Comp
-L Device:R_Small_US R?
+L Device:R_Small_US R13
 U 1 1 63FAA771
 P 3150 2700
-F 0 "R?" V 2945 2700 50  0000 C CNN
+F 0 "R13" V 2945 2700 50  0000 C CNN
 F 1 "0R" V 3036 2700 50  0000 C CNN
-F 2 "" H 3150 2700 50  0001 C CNN
+F 2 "Resistor_SMD:R_0402_1005Metric" H 3150 2700 50  0001 C CNN
 F 3 "~" H 3150 2700 50  0001 C CNN
 	1    3150 2700
@@
 $EndComp
 $Comp
-L Device:C_Small C?
+L Device:C_Small C32
 U 1 1 63FAAE46
 P 2900 3050
-F 0 "C?" H 2808 3004 50  0000 R CNN
+F 0 "C32" H 2808 3004 50  0000 R CNN
 F 1 "NP" H 2808 3095 50  0000 R CNN
-F 2 "" H 2900 3050 50  0001 C CNN
+F 2 "Capacitor_SMD:C_0603_1608Metric" H 2900 3050 50  0001 C CNN
 F 3 "~" H 2900 3050 50  0001 C CNN
 	1    2900 3050
@@
 $EndComp
 $Comp
-L Device:C_Small C?
+L Device:C_Small C33
 U 1 1 63FAB640
 P 3400 3050
-F 0 "C?" H 3308 3004 50  0000 R CNN
+F 0 "C33" H 3308 3004 50  0000 R CNN
 F 1 "NP" H 3308 3095 50  0000 R CNN
-F 2 "" H 3400 3050 50  0001 C CNN
+F 2 "Capacitor_SMD:C_0603_1608Metric" H 3400 3050 50  0001 C CNN
 F 3 "~" H 3400 3050 50  0001 C CNN
 	1    3400 3050
@@
 	3400 2700 3900 2700
 $Comp
-L power:GND #PWR?
+L power:GND #PWR0140
 U 1 1 63FACB4D
 P 2900 3450
-F 0 "#PWR?" H 2900 3200 50  0001 C CNN
+F 0 "#PWR0140" H 2900 3200 50  0001 C CNN
 F 1 "GND" H 2905 3277 50  0000 C CNN
 F 2 "" H 2900 3450 50  0001 C CNN
@@
 $EndComp
 $Comp
-L power:GND #PWR?
+L power:GND #PWR0141
 U 1 1 63FACC7B
 P 3400 3450
-F 0 "#PWR?" H 3400 3200 50  0001 C CNN
+F 0 "#PWR0141" H 3400 3200 50  0001 C CNN
 F 1 "GND" H 3405 3277 50  0000 C CNN
 F 2 "" H 3400 3450 50  0001 C CNN
@@
 $EndComp
 $Comp
-L Device:Antenna AE?
+L Device:Antenna AE3
 U 1 1 63FACFB3
 P 3900 2250
-F 0 "AE?" H 3980 2239 50  0000 L CNN
+F 0 "AE3" H 3980 2239 50  0000 L CNN
 F 1 "Antenna" H 3980 2148 50  0000 L CNN
 F 2 "" H 3900 2250 50  0001 C CNN
@@
 Text HLabel 2400 2700 0    50   Input ~ 0
 ANT_WIFI
-Text Notes 800  1200 0    50   ~ 0
+Text Notes 1350 1450 0    50   ~ 0
 NP = Not Populated\n0R = 0 ohm resitor (jumped)
 Text Notes 2400 2000 0    98   ~ 0
 WIFI
 $Comp
-L Device:R_Small_US R?
+L Device:R_Small_US R14
 U 1 1 63FB1682
 P 6650 2700
-F 0 "R?" V 6445 2700 50  0000 C CNN
+F 0 "R14" V 6445 2700 50  0000 C CNN
 F 1 "0R" V 6536 2700 50  0000 C CNN
-F 2 "" H 6650 2700 50  0001 C CNN
+F 2 "Resistor_SMD:R_0402_1005Metric" H 6650 2700 50  0001 C CNN
 F 3 "~" H 6650 2700 50  0001 C CNN
 	1    6650 2700
@@
 $EndComp
 $Comp
-L Device:C_Small C?
+L Device:C_Small C34
 U 1 1 63FB1688
 P 6400 3050
-F 0 "C?" H 6308 3004 50  0000 R CNN
+F 0 "C34" H 6308 3004 50  0000 R CNN
 F 1 "NP" H 6308 3095 50  0000 R CNN
-F 2 "" H 6400 3050 50  0001 C CNN
+F 2 "Capacitor_SMD:C_0603_1608Metric" H 6400 3050 50  0001 C CNN
 F 3 "~" H 6400 3050 50  0001 C CNN
 	1    6400 3050
@@
 $EndComp
 $Comp
-L Device:C_Small C?
+L Device:C_Small C35
 U 1 1 63FB168E
 P 6900 3050
-F 0 "C?" H 6808 3004 50  0000 R CNN
+F 0 "C35" H 6808 3004 50  0000 R CNN
 F 1 "NP" H 6808 3095 50  0000 R CNN
-F 2 "" H 6900 3050 50  0001 C CNN
+F 2 "Capacitor_SMD:C_0603_1608Metric" H 6900 3050 50  0001 C CNN
 F 3 "~" H 6900 3050 50  0001 C CNN
 	1    6900 3050
@@
 	6900 2700 7050 2700
 $Comp
-L power:GND #PWR?
+L power:GND #PWR0142
 U 1 1 63FB169F
 P 6400 3450
-F 0 "#PWR?" H 6400 3200 50  0001 C CNN
+F 0 "#PWR0142" H 6400 3200 50  0001 C CNN
 F 1 "GND" H 6405 3277 50  0000 C CNN
 F 2 "" H 6400 3450 50  0001 C CNN
@@
 $EndComp
 $Comp
-L power:GND #PWR?
+L power:GND #PWR0143
 U 1 1 63FB16A5
 P 6900 3450
-F 0 "#PWR?" H 6900 3200 50  0001 C CNN
+F 0 "#PWR0143" H 6900 3200 50  0001 C CNN
 F 1 "GND" H 6905 3277 50  0000 C CNN
 F 2 "" H 6900 3450 50  0001 C CNN
@@
 GNSS\n
 $Comp
-L Device:R_Small_US R?
+L Device:R_Small_US R11
 U 1 1 63FDE22B
 P 2450 5000
-F 0 "R?" V 2245 5000 50  0000 C CNN
+F 0 "R11" V 2245 5000 50  0000 C CNN
 F 1 "0R" V 2336 5000 50  0000 C CNN
-F 2 "" H 2450 5000 50  0001 C CNN
+F 2 "Resistor_SMD:R_0402_1005Metric" H 2450 5000 50  0001 C CNN
 F 3 "~" H 2450 5000 50  0001 C CNN
 	1    2450 5000
@@
 $EndComp
 $Comp
-L Device:C_Small C?
+L Device:C_Small C28
 U 1 1 63FDE231
 P 2200 5350
-F 0 "C?" H 2108 5304 50  0000 R CNN
+F 0 "C28" H 2108 5304 50  0000 R CNN
 F 1 "NP" H 2108 5395 50  0000 R CNN
-F 2 "" H 2200 5350 50  0001 C CNN
+F 2 "Capacitor_SMD:C_0603_1608Metric" H 2200 5350 50  0001 C CNN
 F 3 "~" H 2200 5350 50  0001 C CNN
 	1    2200 5350
@@
 $EndComp
 $Comp
-L Device:C_Small C?
+L Device:C_Small C30
 U 1 1 63FDE237
 P 2700 5350
-F 0 "C?" H 2608 5304 50  0000 R CNN
+F 0 "C30" H 2608 5304 50  0000 R CNN
 F 1 "NP" H 2608 5395 50  0000 R CNN
-F 2 "" H 2700 5350 50  0001 C CNN
+F 2 "Capacitor_SMD:C_0603_1608Metric" H 2700 5350 50  0001 C CNN
 F 3 "~" H 2700 5350 50  0001 C CNN
 	1    2700 5350
@@
 	2700 5000 3200 5000
 $Comp
-L power:GND #PWR?
+L power:GND #PWR0144
 U 1 1 63FDE248
 P 2200 5750
-F 0 "#PWR?" H 2200 5500 50  0001 C CNN
+F 0 "#PWR0144" H 2200 5500 50  0001 C CNN
 F 1 "GND" H 2205 5577 50  0000 C CNN
 F 2 "" H 2200 5750 50  0001 C CNN
@@
 $EndComp
 $Comp
-L power:GND #PWR?
+L power:GND #PWR0145
 U 1 1 63FDE24E
 P 2700 5750
-F 0 "#PWR?" H 2700 5500 50  0001 C CNN
+F 0 "#PWR0145" H 2700 5500 50  0001 C CNN
 F 1 "GND" H 2705 5577 50  0000 C CNN
 F 2 "" H 2700 5750 50  0001 C CNN
@@
 $EndComp
 $Comp
-L Device:Antenna AE?
+L Device:Antenna AE1
 U 1 1 63FDE254
 P 3200 4550
-F 0 "AE?" H 3280 4539 50  0000 L CNN
+F 0 "AE1" H 3280 4539 50  0000 L CNN
 F 1 "Antenna" H 3280 4448 50  0000 L CNN
 F 2 "" H 3200 4550 50  0001 C CNN
@@
 MAIN
 $Comp
-L Device:R_Small_US R?
+L Device:R_Small_US R12
 U 1 1 63FE04A1
 P 2450 6200
-F 0 "R?" V 2245 6200 50  0000 C CNN
+F 0 "R12" V 2245 6200 50  0000 C CNN
 F 1 "0R" V 2336 6200 50  0000 C CNN
-F 2 "" H 2450 6200 50  0001 C CNN
+F 2 "Resistor_SMD:R_0402_1005Metric" H 2450 6200 50  0001 C CNN
 F 3 "~" H 2450 6200 50  0001 C CNN
 	1    2450 6200
@@
 $EndComp
 $Comp
-L Device:C_Small C?
+L Device:C_Small C29
 U 1 1 63FE04A7
 P 2200 6550
-F 0 "C?" H 2108 6504 50  0000 R CNN
+F 0 "C29" H 2108 6504 50  0000 R CNN
 F 1 "NP" H 2108 6595 50  0000 R CNN
-F 2 "" H 2200 6550 50  0001 C CNN
+F 2 "Capacitor_SMD:C_0603_1608Metric" H 2200 6550 50  0001 C CNN
 F 3 "~" H 2200 6550 50  0001 C CNN
 	1    2200 6550
@@
 $EndComp
 $Comp
-L Device:C_Small C?
+L Device:C_Small C31
 U 1 1 63FE04AD
 P 2700 6550
-F 0 "C?" H 2608 6504 50  0000 R CNN
+F 0 "C31" H 2608 6504 50  0000 R CNN
 F 1 "NP" H 2608 6595 50  0000 R CNN
-F 2 "" H 2700 6550 50  0001 C CNN
+F 2 "Capacitor_SMD:C_0603_1608Metric" H 2700 6550 50  0001 C CNN
 F 3 "~" H 2700 6550 50  0001 C CNN
 	1    2700 6550
@@
 	2700 6200 3200 6200
 $Comp
-L power:GND #PWR?
+L power:GND #PWR0146
 U 1 1 63FE04BE
 P 2200 6950
-F 0 "#PWR?" H 2200 6700 50  0001 C CNN
+F 0 "#PWR0146" H 2200 6700 50  0001 C CNN
 F 1 "GND" H 2205 6777 50  0000 C CNN
 F 2 "" H 2200 6950 50  0001 C CNN
@@
 $EndComp
 $Comp
-L power:GND #PWR?
+L power:GND #PWR0147
 U 1 1 63FE04C4
 P 2700 6950
-F 0 "#PWR?" H 2700 6700 50  0001 C CNN
+F 0 "#PWR0147" H 2700 6700 50  0001 C CNN
 F 1 "GND" H 2705 6777 50  0000 C CNN
 F 2 "" H 2700 6950 50  0001 C CNN
@@
 $EndComp
 $Comp
-L Device:Antenna AE?
+L Device:Antenna AE2
 U 1 1 63FE04CA
 P 3200 5750
-F 0 "AE?" H 3280 5739 50  0000 L CNN
+F 0 "AE2" H 3280 5739 50  0000 L CNN
 F 1 "Antenna" H 3280 5648 50  0000 L CNN
 F 2 "" H 3200 5750 50  0001 C CNN
@@
 ANT_DRX
 $Comp
-L Device:C_Small C?
+L Device:C_Small C36
 U 1 1 63FED24D
 P 7150 2700
-F 0 "C?" V 7379 2700 50  0000 C CNN
+F 0 "C36" V 7379 2700 50  0000 C CNN
 F 1 "NP" V 7288 2700 50  0000 C CNN
-F 2 "" H 7150 2700 50  0001 C CNN
+F 2 "Capacitor_SMD:C_0603_1608Metric" H 7150 2700 50  0001 C CNN
 F 3 "~" H 7150 2700 50  0001 C CNN
 	1    7150 2700
@@
 	7250 2700 7400 2700
 $Comp
-L Device:Antenna AE?
+L Device:Antenna AE4
 U 1 1 63FB16AB
 P 7400 2250
-F 0 "AE?" H 7480 2239 50  0000 L CNN
+F 0 "AE4" H 7480 2239 50  0000 L CNN
 F 1 "Antenna" H 7480 2148 50  0000 L CNN
 F 2 "" H 7400 2250 50  0001 C CNN
@@
 	1    0    0    -1
 $EndComp
+Text Notes 5050 3300 0    50   ~ 0
+PI antenna circuits\nDon't place caps, leave for \nfuture tuning capabilities.
 $EndSCHEMATC

Commit message: Updated schematics, started working on board layout
Parts:
- C32: renamed from C28; footprint Capacitor_SMD:C_0603_1608Metric -> Capacitor_SMD:C_0805_2012Metric
- C33: renamed from C29; footprint Capacitor_SMD:C_0603_1608Metric -> Capacitor_SMD:C_0805_2012Metric
- C34: renamed from C30; footprint Capacitor_SMD:C_0603_1608Metric -> Capacitor_SMD:C_0805_2012Metric
- C35: renamed from C31; footprint Capacitor_SMD:C_0603_1608Metric -> Capacitor_SMD:C_0805_2012Metric
- C36: renamed from C32; footprint Capacitor_SMD:C_0603_1608Metric -> Capacitor_SMD:C_0805_2012Metric
- C37: renamed from C33; footprint Capacitor_SMD:C_0603_1608Metric -> Capacitor_SMD:C_0805_2012Metric
- C38: renamed from C34; footprint Capacitor_SMD:C_0603_1608Metric -> Capacitor_SMD:C_0805_2012Metric
- C39: renamed from C35; footprint Capacitor_SMD:C_0603_1608Metric -> Capacitor_SMD:C_0805_2012Metric
- C40: renamed from C36; footprint Capacitor_SMD:C_0603_1608Metric -> Capacitor_SMD:C_0805_2012Metric
- renumbered R11 to R16, R12 to R17, R13 to R18, R14 to R19
Changed lines of the file:
@@
 $Descr A4 11693 8268
 encoding utf-8
-Sheet 9 13
+Sheet 8 14
 Title "0x0A SmartPhone"
 Date "2022-09-01"
@@
 $EndDescr
 $Comp
-L Device:R_Small_US R13
+L Device:R_Small_US R18
 U 1 1 63FAA771
 P 3150 2700
-F 0 "R13" V 2945 2700 50  0000 C CNN
+F 0 "R18" V 2945 2700 50  0000 C CNN
 F 1 "0R" V 3036 2700 50  0000 C CNN
 F 2 "Resistor_SMD:R_0402_1005Metric" H 3150 2700 50  0001 C CNN
@@
 $EndComp
 $Comp
-L Device:C_Small C32
+L Device:C_Small C36
 U 1 1 63FAAE46
 P 2900 3050
-F 0 "C32" H 2808 3004 50  0000 R CNN
+F 0 "C36" H 2808 3004 50  0000 R CNN
 F 1 "NP" H 2808 3095 50  0000 R CNN
-F 2 "Capacitor_SMD:C_0603_1608Metric" H 2900 3050 50  0001 C CNN
+F 2 "Capacitor_SMD:C_0805_2012Metric" H 2900 3050 50  0001 C CNN
 F 3 "~" H 2900 3050 50  0001 C CNN
 	1    2900 3050
@@
 $EndComp
 $Comp
-L Device:C_Small C33
+L Device:C_Small C37
 U 1 1 63FAB640
 P 3400 3050
-F 0 "C33" H 3308 3004 50  0000 R CNN
+F 0 "C37" H 3308 3004 50  0000 R CNN
 F 1 "NP" H 3308 3095 50  0000 R CNN
-F 2 "Capacitor_SMD:C_0603_1608Metric" H 3400 3050 50  0001 C CNN
+F 2 "Capacitor_SMD:C_0805_2012Metric" H 3400 3050 50  0001 C CNN
 F 3 "~" H 3400 3050 50  0001 C CNN
 	1    3400 3050
@@
 	3400 2700 3900 2700
 $Comp
-L power:GND #PWR0140
+L power:GND #PWR050
 U 1 1 63FACB4D
 P 2900 3450
-F 0 "#PWR0140" H 2900 3200 50  0001 C CNN
+F 0 "#PWR050" H 2900 3200 50  0001 C CNN
 F 1 "GND" H 2905 3277 50  0000 C CNN
 F 2 "" H 2900 3450 50  0001 C CNN
@@
 $EndComp
 $Comp
-L power:GND #PWR0141
+L power:GND #PWR051
 U 1 1 63FACC7B
 P 3400 3450
-F 0 "#PWR0141" H 3400 3200 50  0001 C CNN
+F 0 "#PWR051" H 3400 3200 50  0001 C CNN
 F 1 "GND" H 3405 3277 50  0000 C CNN
 F 2 "" H 3400 3450 50  0001 C CNN
@@
 WIFI
 $Comp
-L Device:R_Small_US R14
+L Device:R_Small_US R19
 U 1 1 63FB1682
 P 6650 2700
-F 0 "R14" V 6445 2700 50  0000 C CNN
+F 0 "R19" V 6445 2700 50  0000 C CNN
 F 1 "0R" V 6536 2700 50  0000 C CNN
 F 2 "Resistor_SMD:R_0402_1005Metric" H 6650 2700 50  0001 C CNN
@@
 $EndComp
 $Comp
-L Device:C_Small C34
+L Device:C_Small C38
 U 1 1 63FB1688
 P 6400 3050
-F 0 "C34" H 6308 3004 50  0000 R CNN
+F 0 "C38" H 6308 3004 50  0000 R CNN
 F 1 "NP" H 6308 3095 50  0000 R CNN
-F 2 "Capacitor_SMD:C_0603_1608Metric" H 6400 3050 50  0001 C CNN
+F 2 "Capacitor_SMD:C_0805_2012Metric" H 6400 3050 50  0001 C CNN
 F 3 "~" H 6400 3050 50  0001 C CNN
 	1    6400 3050
@@
 $EndComp
 $Comp
-L Device:C_Small C35
+L Device:C_Small C39
 U 1 1 63FB168E
 P 6900 3050
-F 0 "C35" H 6808 3004 50  0000 R CNN
+F 0 "C39" H 6808 3004 50  0000 R CNN
 F 1 "NP" H 6808 3095 50  0000 R CNN
-F 2 "Capacitor_SMD:C_0603_1608Metric" H 6900 3050 50  0001 C CNN
+F 2 "Capacitor_SMD:C_0805_2012Metric" H 6900 3050 50  0001 C CNN
 F 3 "~" H 6900 3050 50  0001 C CNN
 	1    6900 3050
@@
 	6900 2700 7050 2700
 $Comp
-L power:GND #PWR0142
+L power:GND #PWR052
 U 1 1 63FB169F
 P 6400 3450
-F 0 "#PWR0142" H 6400 3200 50  0001 C CNN
+F 0 "#PWR052" H 6400 3200 50  0001 C CNN
 F 1 "GND" H 6405 3277 50  0000 C CNN
 F 2 "" H 6400 3450 50  0001 C CNN
@@
 $EndComp
 $Comp
-L power:GND #PWR0143
+L power:GND #PWR053
 U 1 1 63FB16A5
 P 6900 3450
-F 0 "#PWR0143" H 6900 3200 50  0001 C CNN
+F 0 "#PWR053" H 6900 3200 50  0001 C CNN
 F 1 "GND" H 6905 3277 50  0000 C CNN
 F 2 "" H 6900 3450 50  0001 C CNN
@@
 GNSS\n
 $Comp
-L Device:R_Small_US R11
+L Device:R_Small_US R16
 U 1 1 63FDE22B
 P 2450 5000
-F 0 "R11" V 2245 5000 50  0000 C CNN
+F 0 "R16" V 2245 5000 50  0000 C CNN
 F 1 "0R" V 2336 5000 50  0000 C CNN
 F 2 "Resistor_SMD:R_0402_1005Metric" H 2450 5000 50  0001 C CNN
@@
 $EndComp
 $Comp
-L Device:C_Small C28
+L Device:C_Small C32
 U 1 1 63FDE231
 P 2200 5350
-F 0 "C28" H 2108 5304 50  0000 R CNN
+F 0 "C32" H 2108 5304 50  0000 R CNN
 F 1 "NP" H 2108 5395 50  0000 R CNN
-F 2 "Capacitor_SMD:C_0603_1608Metric" H 2200 5350 50  0001 C CNN
+F 2 "Capacitor_SMD:C_0805_2012Metric" H 2200 5350 50  0001 C CNN
 F 3 "~" H 2200 5350 50  0001 C CNN
 	1    2200 5350
@@
 $EndComp
 $Comp
-L Device:C_Small C30
+L Device:C_Small C34
 U 1 1 63FDE237
 P 2700 5350
-F 0 "C30" H 2608 5304 50  0000 R CNN
+F 0 "C34" H 2608 5304 50  0000 R CNN
 F 1 "NP" H 2608 5395 50  0000 R CNN
-F 2 "Capacitor_SMD:C_0603_1608Metric" H 2700 5350 50  0001 C CNN
+F 2 "Capacitor_SMD:C_0805_2012Metric" H 2700 5350 50  0001 C CNN
 F 3 "~" H 2700 5350 50  0001 C CNN
 	1    2700 5350
@@
 	2700 5000 3200 5000
 $Comp
-L power:GND #PWR0144
+L power:GND #PWR046
 U 1 1 63FDE248
 P 2200 5750
-F 0 "#PWR0144" H 2200 5500 50  0001 C CNN
+F 0 "#PWR046" H 2200 5500 50  0001 C CNN
 F 1 "GND" H 2205 5577 50  0000 C CNN
 F 2 "" H 2200 5750 50  0001 C CNN
@@
 $EndComp
 $Comp
-L power:GND #PWR0145
+L power:GND #PWR048
 U 1 1 63FDE24E
 P 2700 5750
-F 0 "#PWR0145" H 2700 5500 50  0001 C CNN
+F 0 "#PWR048" H 2700 5500 50  0001 C CNN
 F 1 "GND" H 2705 5577 50  0000 C CNN
 F 2 "" H 2700 5750 50  0001 C CNN
@@
 MAIN
 $Comp
-L Device:R_Small_US R12
+L Device:R_Small_US R17
 U 1 1 63FE04A1
 P 2450 6200
-F 0 "R12" V 2245 6200 50  0000 C CNN
+F 0 "R17" V 2245 6200 50  0000 C CNN
 F 1 "0R" V 2336 6200 50  0000 C CNN
 F 2 "Resistor_SMD:R_0402_1005Metric" H 2450 6200 50  0001 C CNN
@@
 $EndComp
 $Comp
-L Device:C_Small C29
+L Device:C_Small C33
 U 1 1 63FE04A7
 P 2200 6550
-F 0 "C29" H 2108 6504 50  0000 R CNN
+F 0 "C33" H 2108 6504 50  0000 R CNN
 F 1 "NP" H 2108 6595 50  0000 R CNN
-F 2 "Capacitor_SMD:C_0603_1608Metric" H 2200 6550 50  0001 C CNN
+F 2 "Capacitor_SMD:C_0805_2012Metric" H 2200 6550 50  0001 C CNN
 F 3 "~" H 2200 6550 50  0001 C CNN
 	1    2200 6550
@@
 $EndComp
 $Comp
-L Device:C_Small C31
+L Device:C_Small C35
 U 1 1 63FE04AD
 P 2700 6550
-F 0 "C31" H 2608 6504 50  0000 R CNN
+F 0 "C35" H 2608 6504 50  0000 R CNN
 F 1 "NP" H 2608 6595 50  0000 R CNN
-F 2 "Capacitor_SMD:C_0603_1608Metric" H 2700 6550 50  0001 C CNN
+F 2 "Capacitor_SMD:C_0805_2012Metric" H 2700 6550 50  0001 C CNN
 F 3 "~" H 2700 6550 50  0001 C CNN
 	1    2700 6550
@@
 	2700 6200 3200 6200
 $Comp
-L power:GND #PWR0146
+L power:GND #PWR047
 U 1 1 63FE04BE
 P 2200 6950
-F 0 "#PWR0146" H 2200 6700 50  0001 C CNN
+F 0 "#PWR047" H 2200 6700 50  0001 C CNN
 F 1 "GND" H 2205 6777 50  0000 C CNN
 F 2 "" H 2200 6950 50  0001 C CNN
@@
 $EndComp
 $Comp
-L power:GND #PWR0147
+L power:GND #PWR049
 U 1 1 63FE04C4
 P 2700 6950
-F 0 "#PWR0147" H 2700 6700 50  0001 C CNN
+F 0 "#PWR049" H 2700 6700 50  0001 C CNN
 F 1 "GND" H 2705 6777 50  0000 C CNN
 F 2 "" H 2700 6950 50  0001 C CNN
@@
 ANT_DRX
 $Comp
-L Device:C_Small C36
+L Device:C_Small C40
 U 1 1 63FED24D
 P 7150 2700
-F 0 "C36" V 7379 2700 50  0000 C CNN
+F 0 "C40" V 7379 2700 50  0000 C CNN
 F 1 "NP" V 7288 2700 50  0000 C CNN
-F 2 "Capacitor_SMD:C_0603_1608Metric" H 7150 2700 50  0001 C CNN
+F 2 "Capacitor_SMD:C_0805_2012Metric" H 7150 2700 50  0001 C CNN
 F 3 "~" H 7150 2700 50  0001 C CNN
 	1    7150 2700
