File: src/0x0A/buttons.sch (KiCad schematic (older format))
At the start: 9 parts

Commit message: new file:   imgs/better.png 	modified:   src/0x0A/0x0A-cache.lib 	modified:   src/0x0A/0x0A.sch 	modified:   src/0x0A/antenna.sch 	modified:   src/0x0A/audio.sch 	modified:   src/0x0A/buttons.sch 	new file:   src/0x0A/cameras.sch 	modified:   src/0x0A/display.sch 	modified:   src/0x0A/gpio.sch 	modified:   src/0x0A/pwr.sch 	modified:   src/0x0A/sensors.sch 	modified:   src/0x0A/sim.sch 	modified:   src/0x0A/uart.sch 	modified:   src/0x0A/usb.sch 	new file:   src/models/body.obj 	new file:   src/models/phone.FCStd 	new file:   src/models/screen.obj
Added 3D models, integrated front & rear cameras, flash light, reformatting & more
Parts:
- R15, R16, R17: renamed from R?; footprint (none) -> Resistor_SMD:R_0402_1005Metric
- gave numbers to parts that had none: 6
Changed lines of the file:
@@
 $Descr A4 11693 8268
 encoding utf-8
-Sheet 11 12
+Sheet 11 13
 Title "0x0A SmartPhone"
 Date "2022-09-01"
 Rev "1"
 Comp "HackThisPhone.com"
-Comment1 ""
+Comment1 "Designed By @NoahGWood for"
 Comment2 ""
 Comment3 ""
@@
 $EndDescr
 $Comp
-L Connector_Generic:Conn_01x02 J?
+L Connector_Generic:Conn_01x02 J14
 U 1 1 645EFBAA
 P 4500 4500
-F 0 "J?" H 4418 4175 50  0000 C CNN
+F 0 "J14" H 4418 4175 50  0000 C CNN
 F 1 "PWRBTN" H 4418 4266 50  0000 C CNN
 F 2 "" H 4500 4500 50  0001 C CNN
@@
 $EndComp
 $Comp
-L Diode:1.5KExxA D?
+L Diode:1.5KExxA D17
 U 1 1 645EFBB0
 P 5200 4550
-F 0 "D?" V 5154 4629 50  0000 L CNN
+F 0 "D17" V 5154 4629 50  0000 L CNN
 F 1 "?" V 5245 4629 50  0000 L CNN
 F 2 "Diode_THT:D_DO-201AE_P15.24mm_Horizontal" H 5200 4350 50  0001 C CNN
@@
 $EndComp
 $Comp
-L power:GND #PWR?
+L power:GND #PWR0148
 U 1 1 645EFBB6
 P 5200 4700
-F 0 "#PWR?" H 5200 4450 50  0001 C CNN
+F 0 "#PWR0148" H 5200 4450 50  0001 C CNN
 F 1 "GND" H 5205 4527 50  0000 C CNN
 F 2 "" H 5200 4700 50  0001 C CNN
@@
 $EndComp
 $Comp
-L power:GND #PWR?
+L power:GND #PWR0149
 U 1 1 645EFBBC
 P 4700 4700
-F 0 "#PWR?" H 4700 4450 50  0001 C CNN
+F 0 "#PWR0149" H 4700 4450 50  0001 C CNN
 F 1 "GND" H 4705 4527 50  0000 C CNN
 F 2 "" H 4700 4700 50  0001 C CNN
@@
 Connection ~ 5200 4400
 $Comp
-L Device:R_Small_US R?
+L Device:R_Small_US R17
 U 1 1 645EFBC6
 P 5450 4400
-F 0 "R?" V 5245 4400 50  0000 C CNN
+F 0 "R17" V 5245 4400 50  0000 C CNN
 F 1 "1k" V 5336 4400 50  0000 C CNN
-F 2 "" H 5450 4400 50  0001 C CNN
+F 2 "Resistor_SMD:R_0402_1005Metric" H 5450 4400 50  0001 C CNN
 F 3 "~" H 5450 4400 50  0001 C CNN
 	1    5450 4400
@@
 P 4500 3500
 AR Path="/6311B05E/645F6A60" Ref="J?"  Part="1"
-AR Path="/645DE31F/645F6A60" Ref="J?"  Part="1"
-F 0 "J?" H 4418 3175 50  0000 C CNN
+AR Path="/645DE31F/645F6A60" Ref="J13"  Part="1"
+F 0 "J13" H 4418 3175 50  0000 C CNN
 F 1 "VOL+" H 4418 3266 50  0000 C CNN
 F 2 "" H 4500 3500 50  0001 C CNN
@@
 $EndComp
 $Comp
-L Diode:1.5KExxA D?
+L Diode:1.5KExxA D16
 U 1 1 645F6A66
 P 5200 3550
-F 0 "D?" V 5154 3629 50  0000 L CNN
+F 0 "D16" V 5154 3629 50  0000 L CNN
 F 1 "?" V 5245 3629 50  0000 L CNN
 F 2 "Diode_THT:D_DO-201AE_P15.24mm_Horizontal" H 5200 3350 50  0001 C CNN
@@
 $EndComp
 $Comp
-L power:GND #PWR?
+L power:GND #PWR0150
 U 1 1 645F6A6C
 P 5200 3700
-F 0 "#PWR?" H 5200 3450 50  0001 C CNN
+F 0 "#PWR0150" H 5200 3450 50  0001 C CNN
 F 1 "GND" H 5205 3527 50  0000 C CNN
 F 2 "" H 5200 3700 50  0001 C CNN
@@
 $EndComp
 $Comp
-L power:GND #PWR?
+L power:GND #PWR0151
 U 1 1 645F6A72
 P 4700 3700
-F 0 "#PWR?" H 4700 3450 50  0001 C CNN
+F 0 "#PWR0151" H 4700 3450 50  0001 C CNN
 F 1 "GND" H 4705 3527 50  0000 C CNN
 F 2 "" H 4700 3700 50  0001 C CNN
@@
 Connection ~ 5200 3400
 $Comp
-L Device:R_Small_US R?
+L Device:R_Small_US R16
 U 1 1 645F6A7C
 P 5450 3400
-F 0 "R?" V 5245 3400 50  0000 C CNN
+F 0 "R16" V 5245 3400 50  0000 C CNN
 F 1 "1k" V 5336 3400 50  0000 C CNN
-F 2 "" H 5450 3400 50  0001 C CNN
+F 2 "Resistor_SMD:R_0402_1005Metric" H 5450 3400 50  0001 C CNN
 F 3 "~" H 5450 3400 50  0001 C CNN
 	1    5450 3400
@@
 P 4500 2500
 AR Path="/6311B05E/645F91B7" Ref="J?"  Part="1"
-AR Path="/645DE31F/645F91B7" Ref="J?"  Part="1"
-F 0 "J?" H 4418 2175 50  0000 C CNN
+AR Path="/645DE31F/645F91B7" Ref="J12"  Part="1"
+F 0 "J12" H 4418 2175 50  0000 C CNN
 F 1 "VOL-" H 4418 2266 50  0000 C CNN
 F 2 "" H 4500 2500 50  0001 C CNN
@@
 $EndComp
 $Comp
-L Diode:1.5KExxA D?
+L Diode:1.5KExxA D15
 U 1 1 645F91BD
 P 5200 2550
-F 0 "D?" V 5154 2629 50  0000 L CNN
+F 0 "D15" V 5154 2629 50  0000 L CNN
 F 1 "?" V 5245 2629 50  0000 L CNN
 F 2 "Diode_THT:D_DO-201AE_P15.24mm_Horizontal" H 5200 2350 50  0001 C CNN
@@
 $EndComp
 $Comp
-L power:GND #PWR?
+L power:GND #PWR0152
 U 1 1 645F91C3
 P 5200 2700
-F 0 "#PWR?" H 5200 2450 50  0001 C CNN
+F 0 "#PWR0152" H 5200 2450 50  0001 C CNN
 F 1 "GND" H 5205 2527 50  0000 C CNN
 F 2 "" H 5200 2700 50  0001 C CNN
@@
 $EndComp
 $Comp
-L power:GND #PWR?
+L power:GND #PWR0153
 U 1 1 645F91C9
 P 4700 2700
-F 0 "#PWR?" H 4700 2450 50  0001 C CNN
+F 0 "#PWR0153" H 4700 2450 50  0001 C CNN
 F 1 "GND" H 4705 2527 50  0000 C CNN
 F 2 "" H 4700 2700 50  0001 C CNN
@@
 Connection ~ 5200 2400
 $Comp
-L Device:R_Small_US R?
+L Device:R_Small_US R15
 U 1 1 645F91D3
 P 5450 2400
-F 0 "R?" V 5245 2400 50  0000 C CNN
+F 0 "R15" V 5245 2400 50  0000 C CNN
 F 1 "1k" V 5336 2400 50  0000 C CNN
-F 2 "" H 5450 2400 50  0001 C CNN
+F 2 "Resistor_SMD:R_0402_1005Metric" H 5450 2400 50  0001 C CNN
 F 3 "~" H 5450 2400 50  0001 C CNN
 	1    5450 2400

Commit message: Updated schematics, started working on board layout
Parts:
- added D20: ?, Diode_THT:D_DO-201AE_P15.24mm_Horizontal, symbol Diode:1.5KExxA
- added R23: 10K, Resistor_SMD:R_0402_1005Metric, symbol Device:R_Small_US
- added SW1: USB_BOOT, symbol Switch:SW_Push
- renumbered D15 to D17, D16 to D18, D17 to D19, J12 to J13, J13 to J14, J14 to J15, R15 to R20, R16 to R21, R17 to R22
Connections:
- net GND: now also D20.2 (A2)
- new net: R23.2, SW1.2
- new net LDO5_1P8: R23.1
- new net USB_BOOT: D20.1 (A1), SW1.1
Changed lines of the file:
@@
 $Descr A4 11693 8268
 encoding utf-8
-Sheet 11 13
+Sheet 9 14
 Title "0x0A SmartPhone"
 Date "2022-09-01"
@@
 $EndDescr
 $Comp
-L Connector_Generic:Conn_01x02 J14
+L Connector_Generic:Conn_01x02 J15
 U 1 1 645EFBAA
 P 4500 4500
-F 0 "J14" H 4418 4175 50  0000 C CNN
+F 0 "J15" H 4418 4175 50  0000 C CNN
 F 1 "PWRBTN" H 4418 4266 50  0000 C CNN
 F 2 "" H 4500 4500 50  0001 C CNN
@@
 $EndComp
 $Comp
-L Diode:1.5KExxA D17
+L Diode:1.5KExxA D19
 U 1 1 645EFBB0
 P 5200 4550
-F 0 "D17" V 5154 4629 50  0000 L CNN
+F 0 "D19" V 5154 4629 50  0000 L CNN
 F 1 "?" V 5245 4629 50  0000 L CNN
 F 2 "Diode_THT:D_DO-201AE_P15.24mm_Horizontal" H 5200 4350 50  0001 C CNN
@@
 $EndComp
 $Comp
-L power:GND #PWR0148
+L power:GND #PWR059
 U 1 1 645EFBB6
 P 5200 4700
-F 0 "#PWR0148" H 5200 4450 50  0001 C CNN
+F 0 "#PWR059" H 5200 4450 50  0001 C CNN
 F 1 "GND" H 5205 4527 50  0000 C CNN
 F 2 "" H 5200 4700 50  0001 C CNN
@@
 $EndComp
 $Comp
-L power:GND #PWR0149
+L power:GND #PWR056
 U 1 1 645EFBBC
 P 4700 4700
-F 0 "#PWR0149" H 4700 4450 50  0001 C CNN
+F 0 "#PWR056" H 4700 4450 50  0001 C CNN
 F 1 "GND" H 4705 4527 50  0000 C CNN
 F 2 "" H 4700 4700 50  0001 C CNN
@@
 Connection ~ 5200 4400
 $Comp
-L Device:R_Small_US R17
+L Device:R_Small_US R22
 U 1 1 645EFBC6
 P 5450 4400
-F 0 "R17" V 5245 4400 50  0000 C CNN
+F 0 "R22" V 5245 4400 50  0000 C CNN
 F 1 "1k" V 5336 4400 50  0000 C CNN
 F 2 "Resistor_SMD:R_0402_1005Metric" H 5450 4400 50  0001 C CNN
@@
 P 4500 3500
 AR Path="/6311B05E/645F6A60" Ref="J?"  Part="1"
-AR Path="/645DE31F/645F6A60" Ref="J13"  Part="1"
-F 0 "J13" H 4418 3175 50  0000 C CNN
+AR Path="/645DE31F/645F6A60" Ref="J14"  Part="1"
+F 0 "J14" H 4418 3175 50  0000 C CNN
 F 1 "VOL+" H 4418 3266 50  0000 C CNN
 F 2 "" H 4500 3500 50  0001 C CNN
@@
 $EndComp
 $Comp
-L Diode:1.5KExxA D16
+L Diode:1.5KExxA D18
 U 1 1 645F6A66
 P 5200 3550
-F 0 "D16" V 5154 3629 50  0000 L CNN
+F 0 "D18" V 5154 3629 50  0000 L CNN
 F 1 "?" V 5245 3629 50  0000 L CNN
 F 2 "Diode_THT:D_DO-201AE_P15.24mm_Horizontal" H 5200 3350 50  0001 C CNN
@@
 $EndComp
 $Comp
-L power:GND #PWR0150
+L power:GND #PWR058
 U 1 1 645F6A6C
 P 5200 3700
-F 0 "#PWR0150" H 5200 3450 50  0001 C CNN
+F 0 "#PWR058" H 5200 3450 50  0001 C CNN
 F 1 "GND" H 5205 3527 50  0000 C CNN
 F 2 "" H 5200 3700 50  0001 C CNN
@@
 $EndComp
 $Comp
-L power:GND #PWR0151
+L power:GND #PWR055
 U 1 1 645F6A72
 P 4700 3700
-F 0 "#PWR0151" H 4700 3450 50  0001 C CNN
+F 0 "#PWR055" H 4700 3450 50  0001 C CNN
 F 1 "GND" H 4705 3527 50  0000 C CNN
 F 2 "" H 4700 3700 50  0001 C CNN
@@
 Connection ~ 5200 3400
 $Comp
-L Device:R_Small_US R16
+L Device:R_Small_US R21
 U 1 1 645F6A7C
 P 5450 3400
-F 0 "R16" V 5245 3400 50  0000 C CNN
+F 0 "R21" V 5245 3400 50  0000 C CNN
 F 1 "1k" V 5336 3400 50  0000 C CNN
 F 2 "Resistor_SMD:R_0402_1005Metric" H 5450 3400 50  0001 C CNN
@@
 P 4500 2500
 AR Path="/6311B05E/645F91B7" Ref="J?"  Part="1"
-AR Path="/645DE31F/645F91B7" Ref="J12"  Part="1"
-F 0 "J12" H 4418 2175 50  0000 C CNN
+AR Path="/645DE31F/645F91B7" Ref="J13"  Part="1"
+F 0 "J13" H 4418 2175 50  0000 C CNN
 F 1 "VOL-" H 4418 2266 50  0000 C CNN
 F 2 "" H 4500 2500 50  0001 C CNN
@@
 $EndComp
 $Comp
-L Diode:1.5KExxA D15
+L Diode:1.5KExxA D17
 U 1 1 645F91BD
 P 5200 2550
-F 0 "D15" V 5154 2629 50  0000 L CNN
+F 0 "D17" V 5154 2629 50  0000 L CNN
 F 1 "?" V 5245 2629 50  0000 L CNN
 F 2 "Diode_THT:D_DO-201AE_P15.24mm_Horizontal" H 5200 2350 50  0001 C CNN
@@
 $EndComp
 $Comp
-L power:GND #PWR0152
+L power:GND #PWR057
 U 1 1 645F91C3
 P 5200 2700
-F 0 "#PWR0152" H 5200 2450 50  0001 C CNN
+F 0 "#PWR057" H 5200 2450 50  0001 C CNN
 F 1 "GND" H 5205 2527 50  0000 C CNN
 F 2 "" H 5200 2700 50  0001 C CNN
@@
 $EndComp
 $Comp
-L power:GND #PWR0153
+L power:GND #PWR054
 U 1 1 645F91C9
 P 4700 2700
-F 0 "#PWR0153" H 4700 2450 50  0001 C CNN
+F 0 "#PWR054" H 4700 2450 50  0001 C CNN
 F 1 "GND" H 4705 2527 50  0000 C CNN
 F 2 "" H 4700 2700 50  0001 C CNN
@@
 Connection ~ 5200 2400
 $Comp
-L Device:R_Small_US R15
+L Device:R_Small_US R20
 U 1 1 645F91D3
 P 5450 2400
-F 0 "R15" V 5245 2400 50  0000 C CNN
+F 0 "R20" V 5245 2400 50  0000 C CNN
 F 1 "1k" V 5336 2400 50  0000 C CNN
 F 2 "Resistor_SMD:R_0402_1005Metric" H 5450 2400 50  0001 C CNN
@@
 Text HLabel 5700 2400 2    50   Input ~ 0
 VOL_DOWN
+Wire Wire Line
+	9100 2050 8950 2050
+$Comp
+L Device:R_Small_US R23
+U 1 1 64611717
+P 8850 2050
+F 0 "R23" V 8645 2050 50  0000 C CNN
+F 1 "10K" V 8736 2050 50  0000 C CNN
+F 2 "Resistor_SMD:R_0402_1005Metric" H 8850 2050 50  0001 C CNN
+F 3 "~" H 8850 2050 50  0001 C CNN
+	1    8850 2050
+	0    1    1    0
+$EndComp
+Text HLabel 9100 2050 2    50   Input ~ 0
+LDO5_1P8
+Wire Wire Line
+	8100 2050 8200 2050
+$Comp
+L Diode:1.5KExxA D20
+U 1 1 6461373D
+P 8100 2200
+F 0 "D20" V 8054 2279 50  0000 L CNN
+F 1 "?" V 8145 2279 50  0000 L CNN
+F 2 "Diode_THT:D_DO-201AE_P15.24mm_Horizontal" H 8100 2000 50  0001 C CNN
+F 3 "https://www.vishay.com/docs/88301/15ke.pdf" H 8050 2200 50  0001 C CNN
+	1    8100 2200
+	0    1    1    0
+$EndComp
+$Comp
+L power:GND #PWR060
+U 1 1 64613743
+P 8100 2350
+F 0 "#PWR060" H 8100 2100 50  0001 C CNN
+F 1 "GND" H 8105 2177 50  0000 C CNN
+F 2 "" H 8100 2350 50  0001 C CNN
+F 3 "" H 8100 2350 50  0001 C CNN
+	1    8100 2350
+	1    0    0    -1
+$EndComp
+$Comp
+L Switch:SW_Push SW1
+U 1 1 64616454
+P 8400 2050
+F 0 "SW1" H 8400 2335 50  0000 C CNN
+F 1 "USB_BOOT" H 8400 2244 50  0000 C CNN
+F 2 "" H 8400 2250 50  0001 C CNN
+F 3 "~" H 8400 2250 50  0001 C CNN
+	1    8400 2050
+	1    0    0    -1
+$EndComp
+Wire Wire Line
+	8600 2050 8750 2050
+Text HLabel 8100 2050 0    50   Input ~ 0
+USB_BOOT
 $EndSCHEMATC
