File: src/0x0A/display.sch (KiCad schematic (older format))
At the start: 16 parts

Commit message: new file:   imgs/better.png 	modified:   src/0x0A/0x0A-cache.lib 	modified:   src/0x0A/0x0A.sch 	modified:   src/0x0A/antenna.sch 	modified:   src/0x0A/audio.sch 	modified:   src/0x0A/buttons.sch 	new file:   src/0x0A/cameras.sch 	modified:   src/0x0A/display.sch 	modified:   src/0x0A/gpio.sch 	modified:   src/0x0A/pwr.sch 	modified:   src/0x0A/sensors.sch 	modified:   src/0x0A/sim.sch 	modified:   src/0x0A/uart.sch 	modified:   src/0x0A/usb.sch 	new file:   src/models/body.obj 	new file:   src/models/phone.FCStd 	new file:   src/models/screen.obj
Added 3D models, integrated front & rear cameras, flash light, reformatting & more
Parts:
- C18, C19, C20, C21, C22: renamed from C?; footprint (none) -> Capacitor_SMD:C_0603_1608Metric
- R7, R8: renamed from R?; footprint (none) -> Resistor_SMD:R_0402_1005Metric
- gave numbers to parts that had none: 9

Commit message: Updated schematics, started working on board layout
Parts:
- removed J6: Conn_2Rows-25Pins, symbol Connector_Generic:Conn_2Rows-25Pins
- removed J7: Conn_01x06, symbol Connector_Generic:Conn_01x06
- added J7: FH26W-25S-0.3SHW(60), SnapEDA Library:HRS_FH26W-25S-0.3SHW(60), symbol FH26W-25S-0.3SHW_60_:FH26W-25S-0.3SHW(60)
- added J8: TF12S-6S-0.5SH(800), SnapEDA Library:HRS_TF12S-6S-0.5SH(800), symbol TF12S-6S-0.5SH_800_:TF12S-6S-0.5SH(800)
- C22: renamed from C18; footprint Capacitor_SMD:C_0603_1608Metric -> Capacitor_SMD:C_0805_2012Metric; LCSC Part # (none) -> C1779
- C23: renamed from C19; footprint Capacitor_SMD:C_0603_1608Metric -> Capacitor_SMD:C_0402_1005Metric; LCSC Part # (none) -> C307331
- C25: renamed from C21; value 4.7uf -> 4.7uF; footprint Capacitor_SMD:C_0603_1608Metric -> Capacitor_SMD:C_0805_2012Metric; LCSC Part # (none) -> C1779
- C26: renamed from C22; footprint Capacitor_SMD:C_0603_1608Metric -> Capacitor_SMD:C_0402_1005Metric; LCSC Part # (none) -> C307331
- J5: renamed from J4; LCSC Part # (none) -> C966916
- J6: renamed from J5; LCSC Part # (none) -> C966916
- renumbered C20 to C24, D8 to D10, D9 to D11, D5 to D7, D6 to D8, D7 to D9, R7 to R12, R8 to R13
Connections:
- net CLKN: now also J7.9
- net CLKP: now also J7.8
- net D0N: now also J7.15
- net D0P: now also J7.14
- net D1N: now also J7.12
- net D1P: now also J7.11
- net D2N: now also J7.6
- net D2P: now also J7.5
- net D3N: now also J7.3
- net D3P: now also J7.2
- net GND: now also J7.1, J7.10, J7.13, J7.16, J7.4, J7.7, J7.S1 (SHIELD), J7.S2 (SHIELD), J8.2
- net INT: now also J8.3
- net IOVDD_1.8V: now also J7.19
- net LCD_ID: now also J7.21
- net LEDA: now also J7.24
- net LEDK: now also J7.23
- net LPTE: now also J7.18
- net RESET: now also J7.17
- net RST: now also J8.4
- net SCL2: now also J8.6
- net SDA2: now also J8.5
- net TP_VCI: now also J8.1
- net VCI_2.8V: now also J7.20
