File: src/0x0A/sensors.sch (KiCad schematic (older format))
At the start: 11 parts

Commit message: new file:   imgs/better.png 	modified:   src/0x0A/0x0A-cache.lib 	modified:   src/0x0A/0x0A.sch 	modified:   src/0x0A/antenna.sch 	modified:   src/0x0A/audio.sch 	modified:   src/0x0A/buttons.sch 	new file:   src/0x0A/cameras.sch 	modified:   src/0x0A/display.sch 	modified:   src/0x0A/gpio.sch 	modified:   src/0x0A/pwr.sch 	modified:   src/0x0A/sensors.sch 	modified:   src/0x0A/sim.sch 	modified:   src/0x0A/uart.sch 	modified:   src/0x0A/usb.sch 	new file:   src/models/body.obj 	new file:   src/models/phone.FCStd 	new file:   src/models/screen.obj
Added 3D models, integrated front & rear cameras, flash light, reformatting & more
Parts:
- C37, C38, C39, C40: renamed from C?; footprint (none) -> Capacitor_SMD:C_0603_1608Metric
- R18, R19, R20, R21, R22: renamed from R?; footprint (none) -> Resistor_SMD:R_0402_1005Metric
- gave numbers to parts that had none: 2
Changed lines of the file:
@@
 $Descr A4 11693 8268
 encoding utf-8
-Sheet 12 12
-Title ""
-Date ""
-Rev ""
-Comp ""
-Comment1 ""
+Sheet 11 13
+Title "0x0A SmartPhone"
+Date "2022-09-01"
+Rev "1"
+Comp "HackThisPhone.com"
+Comment1 "Designed By @NoahGWood for"
 Comment2 ""
 Comment3 ""
@@
 $EndDescr
 $Comp
-L Connector_Generic:Conn_02x04_Counter_Clockwise J?
+L Connector_Generic:Conn_02x04_Counter_Clockwise J15
 U 1 1 64C66F0B
 P 1850 1750
-F 0 "J?" H 1900 2067 50  0000 C CNN
+F 0 "J15" H 1900 2067 50  0000 C CNN
 F 1 "STK3311 (WV|S34)" H 1900 1976 50  0000 C CNN
 F 2 "" H 1850 1750 50  0001 C CNN
@@
 	1    0    0    -1
 $EndComp
-Text HLabel 1650 1650 0    50   Input ~ 0
-SDA
 Text HLabel 2150 1750 2    50   Input ~ 0
 ALS_SDC
@@
 	2600 1950 2150 1950
 $Comp
-L Device:C_Small C?
+L Device:C_Small C37
 U 1 1 64C6A251
 P 2900 1550
-F 0 "C?" H 2992 1596 50  0000 L CNN
+F 0 "C37" H 2992 1596 50  0000 L CNN
 F 1 "4.7uF" H 2992 1505 50  0000 L CNN
-F 2 "" H 2900 1550 50  0001 C CNN
+F 2 "Capacitor_SMD:C_0603_1608Metric" H 2900 1550 50  0001 C CNN
 F 3 "~" H 2900 1550 50  0001 C CNN
 	1    2900 1550
@@
 $EndComp
 $Comp
-L power:GND #PWR?
+L power:GND #PWR0154
 U 1 1 64C6A77D
 P 2900 1950
-F 0 "#PWR?" H 2900 1700 50  0001 C CNN
+F 0 "#PWR0154" H 2900 1700 50  0001 C CNN
 F 1 "GND" H 2905 1777 50  0000 C CNN
 F 2 "" H 2900 1950 50  0001 C CNN
@@
 	2900 1850 2900 1650
 $Comp
-L Device:R_Small_US R?
+L Device:R_Small_US R18
 U 1 1 64C6AF03
 P 1150 1450
-F 0 "R?" H 1218 1496 50  0000 L CNN
+F 0 "R18" H 1218 1496 50  0000 L CNN
 F 1 "10K" H 1218 1405 50  0000 L CNN
-F 2 "" H 1150 1450 50  0001 C CNN
+F 2 "Resistor_SMD:R_0402_1005Metric" H 1150 1450 50  0001 C CNN
 F 3 "~" H 1150 1450 50  0001 C CNN
 	1    1150 1450
@@
 NoConn ~ 1650 1950
 $Comp
-L Device:R_Small_US R?
+L Device:R_Small_US R19
 U 1 1 64C6BB85
 P 1350 2000
-F 0 "R?" H 1418 2046 50  0000 L CNN
+F 0 "R19" H 1418 2046 50  0000 L CNN
 F 1 "NP" H 1418 1955 50  0000 L CNN
-F 2 "" H 1350 2000 50  0001 C CNN
+F 2 "Resistor_SMD:R_0402_1005Metric" H 1350 2000 50  0001 C CNN
 F 3 "~" H 1350 2000 50  0001 C CNN
 	1    1350 2000
@@
 $EndComp
 $Comp
-L power:GND #PWR?
+L power:GND #PWR0155
 U 1 1 64C6BF9A
 P 1350 2100
-F 0 "#PWR?" H 1350 1850 50  0001 C CNN
+F 0 "#PWR0155" H 1350 1850 50  0001 C CNN
 F 1 "GND" H 1355 1927 50  0000 C CNN
 F 2 "" H 1350 2100 50  0001 C CNN
@@
 	3400 2650 450  2650
 $Comp
-L Sensor_Motion:MPU-9250 U?
+L Sensor_Motion:MPU-9250 U2
 U 1 1 64C870BF
 P 3900 6350
-F 0 "U?" H 3900 5361 50  0000 C CNN
+F 0 "U2" H 3900 5361 50  0000 C CNN
 F 1 "MPU-9250" H 3900 5270 50  0000 C CNN
 F 2 "Sensor_Motion:InvenSense_QFN-24_3x3mm_P0.4mm" H 3900 5350 50  0001 C CNN
@@
 FSYNC
 $Comp
-L Device:R_Small_US R?
+L Device:R_Small_US R22
 U 1 1 64CAB88F
 P 2700 6550
-F 0 "R?" V 2495 6550 50  0000 C CNN
+F 0 "R22" V 2495 6550 50  0000 C CNN
 F 1 "NP" V 2586 6550 50  0000 C CNN
-F 2 "" H 2700 6550 50  0001 C CNN
+F 2 "Resistor_SMD:R_0402_1005Metric" H 2700 6550 50  0001 C CNN
 F 3 "~" H 2700 6550 50  0001 C CNN
 	1    2700 6550
@@
 	2800 6550 3000 6550
 $Comp
-L Device:R_Small_US R?
+L Device:R_Small_US R20
 U 1 1 64CAD752
 P 2450 6100
-F 0 "R?" H 2382 6054 50  0000 R CNN
+F 0 "R20" H 2382 6054 50  0000 R CNN
 F 1 "OR" H 2382 6145 50  0000 R CNN
-F 2 "" H 2450 6100 50  0001 C CNN
+F 2 "Resistor_SMD:R_0402_1005Metric" H 2450 6100 50  0001 C CNN
 F 3 "~" H 2450 6100 50  0001 C CNN
 	1    2450 6100
@@
 $EndComp
 $Comp
-L power:GND #PWR?
+L power:GND #PWR0156
 U 1 1 64CADF53
 P 2450 6200
-F 0 "#PWR?" H 2450 5950 50  0001 C CNN
+F 0 "#PWR0156" H 2450 5950 50  0001 C CNN
 F 1 "GND" H 2455 6027 50  0000 C CNN
 F 2 "" H 2450 6200 50  0001 C CNN
@@
 $EndComp
 $Comp
-L Device:C_Small C?
+L Device:C_Small C39
 U 1 1 63122067
 P 4200 5300
-F 0 "C?" H 4292 5346 50  0000 L CNN
+F 0 "C39" H 4292 5346 50  0000 L CNN
 F 1 "100nF" H 4292 5255 50  0000 L CNN
-F 2 "" H 4200 5300 50  0001 C CNN
+F 2 "Capacitor_SMD:C_0603_1608Metric" H 4200 5300 50  0001 C CNN
 F 3 "~" H 4200 5300 50  0001 C CNN
 	1    4200 5300
@@
 $EndComp
 $Comp
-L Device:C_Small C?
+L Device:C_Small C38
 U 1 1 63122448
 P 3600 5300
-F 0 "C?" H 3692 5346 50  0000 L CNN
+F 0 "C38" H 3692 5346 50  0000 L CNN
 F 1 "10nF" H 3692 5255 50  0000 L CNN
-F 2 "" H 3600 5300 50  0001 C CNN
+F 2 "Capacitor_SMD:C_0603_1608Metric" H 3600 5300 50  0001 C CNN
 F 3 "~" H 3600 5300 50  0001 C CNN
 	1    3600 5300
@@
 $EndComp
 $Comp
-L power:GND #PWR?
+L power:GND #PWR0157
 U 1 1 63126D52
 P 4200 5400
-F 0 "#PWR?" H 4200 5150 50  0001 C CNN
+F 0 "#PWR0157" H 4200 5150 50  0001 C CNN
 F 1 "GND" H 4205 5227 50  0000 C CNN
 F 2 "" H 4200 5400 50  0001 C CNN
@@
 $EndComp
 $Comp
-L power:GND #PWR?
+L power:GND #PWR0158
 U 1 1 6312766C
 P 3600 5400
-F 0 "#PWR?" H 3600 5150 50  0001 C CNN
+F 0 "#PWR0158" H 3600 5150 50  0001 C CNN
 F 1 "GND" H 3605 5227 50  0000 C CNN
 F 2 "" H 3600 5400 50  0001 C CNN
@@
 	5100 6550 5100 6700
 $Comp
-L Device:C_Small C?
+L Device:C_Small C40
 U 1 1 6313033A
 P 5100 6800
-F 0 "C?" H 5192 6846 50  0000 L CNN
+F 0 "C40" H 5192 6846 50  0000 L CNN
 F 1 "100nF" H 5192 6755 50  0000 L CNN
-F 2 "" H 5100 6800 50  0001 C CNN
+F 2 "Capacitor_SMD:C_0603_1608Metric" H 5100 6800 50  0001 C CNN
 F 3 "~" H 5100 6800 50  0001 C CNN
 	1    5100 6800
@@
 	5100 6900 5100 7050
 $Comp
-L power:GND #PWR?
+L power:GND #PWR0159
 U 1 1 6313084B
 P 5100 7050
-F 0 "#PWR?" H 5100 6800 50  0001 C CNN
+F 0 "#PWR0159" H 5100 6800 50  0001 C CNN
 F 1 "GND" H 5105 6877 50  0000 C CNN
 F 2 "" H 5100 7050 50  0001 C CNN
@@
 	4600 6750 4600 6650
 $Comp
-L power:GND #PWR?
+L power:GND #PWR0160
 U 1 1 63130F3E
 P 4600 7250
-F 0 "#PWR?" H 4600 7000 50  0001 C CNN
+F 0 "#PWR0160" H 4600 7000 50  0001 C CNN
 F 1 "GND" H 4605 7077 50  0000 C CNN
 F 2 "" H 4600 7250 50  0001 C CNN
@@
 	2750 5050 2750 5700
 $Comp
-L Device:R_Small_US R?
+L Device:R_Small_US R21
 U 1 1 6313BFA4
 P 2550 5700
-F 0 "R?" V 2345 5700 50  0000 C CNN
+F 0 "R21" V 2345 5700 50  0000 C CNN
 F 1 "NP" V 2436 5700 50  0000 C CNN
-F 2 "" H 2550 5700 50  0001 C CNN
+F 2 "Resistor_SMD:R_0402_1005Metric" H 2550 5700 50  0001 C CNN
 F 3 "~" H 2550 5700 50  0001 C CNN
 	1    2550 5700
@@
 Text Notes 4350 4750 2    98   ~ 0
 Gyroscopic/Acceleration Sensor
+Text HLabel 1650 1650 0    50   Input ~ 0
+SDA
 $EndSCHEMATC

Commit message: Updated schematics, started working on board layout
Parts:
- C79: renamed from C37; footprint Capacitor_SMD:C_0603_1608Metric -> Capacitor_SMD:C_0805_2012Metric; LCSC Part # (none) -> C1779
- C80: renamed from C38; footprint Capacitor_SMD:C_0603_1608Metric -> Capacitor_SMD:C_0402_1005Metric; LCSC Part # (none) -> C15195
- C81: renamed from C39; footprint Capacitor_SMD:C_0603_1608Metric -> Capacitor_SMD:C_0402_1005Metric; LCSC Part # (none) -> C307331
- C82: renamed from C40; footprint Capacitor_SMD:C_0603_1608Metric -> Capacitor_SMD:C_0402_1005Metric; LCSC Part # (none) -> C307331
- J20: renamed from J15; footprint (none) -> 0x0A:STK3311
- renumbered R18 to R25, R19 to R26, R20 to R27, R21 to R28, R22 to R29, U2 to U8
Connections:
- net GYRO_SCL is gone; now on net SENSOR_I2C_SCL: U8.23 (SCL/SCLK)
- net SDA is gone; now on net SENSOR_I2C_SDA: J20.1 (Pin_1)
- net ALS_SDA renamed ALS_INT_N
- net ALS_SDC renamed SENSOR_I2C_SCL
- net GYRO_SDA renamed SENSOR_I2C_SDA
Changed lines of the file:
@@
 $Descr A4 11693 8268
 encoding utf-8
-Sheet 11 13
+Sheet 12 14
 Title "0x0A SmartPhone"
 Date "2022-09-01"
@@
 $EndDescr
 $Comp
-L Connector_Generic:Conn_02x04_Counter_Clockwise J15
+L Connector_Generic:Conn_02x04_Counter_Clockwise J20
 U 1 1 64C66F0B
 P 1850 1750
-F 0 "J15" H 1900 2067 50  0000 C CNN
+F 0 "J20" H 1900 2067 50  0000 C CNN
 F 1 "STK3311 (WV|S34)" H 1900 1976 50  0000 C CNN
-F 2 "" H 1850 1750 50  0001 C CNN
+F 2 "0x0A:STK3311" H 1850 1750 50  0001 C CNN
 F 3 "~" H 1850 1750 50  0001 C CNN
 	1    1850 1750
 	1    0    0    -1
 $EndComp
-Text HLabel 2150 1750 2    50   Input ~ 0
-ALS_SDC
 Wire Wire Line
 	1650 1750 1150 1750
@@
 	1150 1750 1150 1550
 Text HLabel 1150 1750 0    50   Input ~ 0
-ALS_SDA
+ALS_INT_N
 Wire Wire Line
 	2150 1650 2350 1650
@@
 	2600 1950 2150 1950
 $Comp
-L Device:C_Small C37
+L Device:C_Small C79
 U 1 1 64C6A251
 P 2900 1550
-F 0 "C37" H 2992 1596 50  0000 L CNN
+F 0 "C79" H 2992 1596 50  0000 L CNN
 F 1 "4.7uF" H 2992 1505 50  0000 L CNN
-F 2 "Capacitor_SMD:C_0603_1608Metric" H 2900 1550 50  0001 C CNN
+F 2 "Capacitor_SMD:C_0805_2012Metric" H 2900 1550 50  0001 C CNN
 F 3 "~" H 2900 1550 50  0001 C CNN
+F 4 "C1779" H 2900 1550 50  0001 C CNN "LCSC Part #"
 	1    2900 1550
 	1    0    0    -1
 $EndComp
 $Comp
-L power:GND #PWR0154
+L power:GND #PWR085
 U 1 1 64C6A77D
 P 2900 1950
-F 0 "#PWR0154" H 2900 1700 50  0001 C CNN
+F 0 "#PWR085" H 2900 1700 50  0001 C CNN
 F 1 "GND" H 2905 1777 50  0000 C CNN
 F 2 "" H 2900 1950 50  0001 C CNN
@@
 	2900 1850 2900 1650
 $Comp
-L Device:R_Small_US R18
+L Device:R_Small_US R25
 U 1 1 64C6AF03
 P 1150 1450
-F 0 "R18" H 1218 1496 50  0000 L CNN
+F 0 "R25" H 1218 1496 50  0000 L CNN
 F 1 "10K" H 1218 1405 50  0000 L CNN
 F 2 "Resistor_SMD:R_0402_1005Metric" H 1150 1450 50  0001 C CNN
@@
 NoConn ~ 1650 1950
 $Comp
-L Device:R_Small_US R19
+L Device:R_Small_US R26
 U 1 1 64C6BB85
 P 1350 2000
-F 0 "R19" H 1418 2046 50  0000 L CNN
+F 0 "R26" H 1418 2046 50  0000 L CNN
 F 1 "NP" H 1418 1955 50  0000 L CNN
 F 2 "Resistor_SMD:R_0402_1005Metric" H 1350 2000 50  0001 C CNN
@@
 $EndComp
 $Comp
-L power:GND #PWR0155
+L power:GND #PWR083
 U 1 1 64C6BF9A
 P 1350 2100
-F 0 "#PWR0155" H 1350 1850 50  0001 C CNN
+F 0 "#PWR083" H 1350 1850 50  0001 C CNN
 F 1 "GND" H 1355 1927 50  0000 C CNN
 F 2 "" H 1350 2100 50  0001 C CNN
@@
 	3400 2650 450  2650
 $Comp
-L Sensor_Motion:MPU-9250 U2
+L Sensor_Motion:MPU-9250 U8
 U 1 1 64C870BF
 P 3900 6350
-F 0 "U2" H 3900 5361 50  0000 C CNN
+F 0 "U8" H 3900 5361 50  0000 C CNN
 F 1 "MPU-9250" H 3900 5270 50  0000 C CNN
 F 2 "Sensor_Motion:InvenSense_QFN-24_3x3mm_P0.4mm" H 3900 5350 50  0001 C CNN
@@
 FSYNC
 $Comp
-L Device:R_Small_US R22
+L Device:R_Small_US R29
 U 1 1 64CAB88F
 P 2700 6550
-F 0 "R22" V 2495 6550 50  0000 C CNN
+F 0 "R29" V 2495 6550 50  0000 C CNN
 F 1 "NP" V 2586 6550 50  0000 C CNN
 F 2 "Resistor_SMD:R_0402_1005Metric" H 2700 6550 50  0001 C CNN
@@
 	2800 6550 3000 6550
 $Comp
-L Device:R_Small_US R20
+L Device:R_Small_US R27
 U 1 1 64CAD752
 P 2450 6100
-F 0 "R20" H 2382 6054 50  0000 R CNN
+F 0 "R27" H 2382 6054 50  0000 R CNN
 F 1 "OR" H 2382 6145 50  0000 R CNN
 F 2 "Resistor_SMD:R_0402_1005Metric" H 2450 6100 50  0001 C CNN
@@
 $EndComp
 $Comp
-L power:GND #PWR0156
+L power:GND #PWR084
 U 1 1 64CADF53
 P 2450 6200
-F 0 "#PWR0156" H 2450 5950 50  0001 C CNN
+F 0 "#PWR084" H 2450 5950 50  0001 C CNN
 F 1 "GND" H 2455 6027 50  0000 C CNN
 F 2 "" H 2450 6200 50  0001 C CNN
@@
 $EndComp
 $Comp
-L Device:C_Small C39
+L Device:C_Small C81
 U 1 1 63122067
 P 4200 5300
-F 0 "C39" H 4292 5346 50  0000 L CNN
+F 0 "C81" H 4292 5346 50  0000 L CNN
 F 1 "100nF" H 4292 5255 50  0000 L CNN
-F 2 "Capacitor_SMD:C_0603_1608Metric" H 4200 5300 50  0001 C CNN
+F 2 "Capacitor_SMD:C_0402_1005Metric" H 4200 5300 50  0001 C CNN
 F 3 "~" H 4200 5300 50  0001 C CNN
+F 4 "C307331" H 4200 5300 50  0001 C CNN "LCSC Part #"
 	1    4200 5300
 	1    0    0    -1
 $EndComp
 $Comp
-L Device:C_Small C38
+L Device:C_Small C80
 U 1 1 63122448
 P 3600 5300
-F 0 "C38" H 3692 5346 50  0000 L CNN
+F 0 "C80" H 3692 5346 50  0000 L CNN
 F 1 "10nF" H 3692 5255 50  0000 L CNN
-F 2 "Capacitor_SMD:C_0603_1608Metric" H 3600 5300 50  0001 C CNN
+F 2 "Capacitor_SMD:C_0402_1005Metric" H 3600 5300 50  0001 C CNN
 F 3 "~" H 3600 5300 50  0001 C CNN
+F 4 "C15195" H 3600 5300 50  0001 C CNN "LCSC Part #"
 	1    3600 5300
 	-1   0    0    -1
 $EndComp
 $Comp
-L power:GND #PWR0157
+L power:GND #PWR087
 U 1 1 63126D52
 P 4200 5400
-F 0 "#PWR0157" H 4200 5150 50  0001 C CNN
+F 0 "#PWR087" H 4200 5150 50  0001 C CNN
 F 1 "GND" H 4205 5227 50  0000 C CNN
 F 2 "" H 4200 5400 50  0001 C CNN
@@
 $EndComp
 $Comp
-L power:GND #PWR0158
+L power:GND #PWR086
 U 1 1 6312766C
 P 3600 5400
-F 0 "#PWR0158" H 3600 5150 50  0001 C CNN
+F 0 "#PWR086" H 3600 5150 50  0001 C CNN
 F 1 "GND" H 3605 5227 50  0000 C CNN
 F 2 "" H 3600 5400 50  0001 C CNN
@@
 	4000 5050 4000 5200
 Connection ~ 4000 5200
-Text HLabel 3200 6050 0    50   Input ~ 0
-GYRO_SDA
-Text HLabel 3200 6250 0    50   Input ~ 0
-GYRO_SCL
 Text HLabel 4600 6050 2    50   Input ~ 0
 GYRO_INT
@@
 	5100 6550 5100 6700
 $Comp
-L Device:C_Small C40
+L Device:C_Small C82
 U 1 1 6313033A
 P 5100 6800
-F 0 "C40" H 5192 6846 50  0000 L CNN
+F 0 "C82" H 5192 6846 50  0000 L CNN
 F 1 "100nF" H 5192 6755 50  0000 L CNN
-F 2 "Capacitor_SMD:C_0603_1608Metric" H 5100 6800 50  0001 C CNN
+F 2 "Capacitor_SMD:C_0402_1005Metric" H 5100 6800 50  0001 C CNN
 F 3 "~" H 5100 6800 50  0001 C CNN
+F 4 "C307331" H 5100 6800 50  0001 C CNN "LCSC Part #"
 	1    5100 6800
 	1    0    0    -1
@@
 	5100 6900 5100 7050
 $Comp
-L power:GND #PWR0159
+L power:GND #PWR089
 U 1 1 6313084B
 P 5100 7050
-F 0 "#PWR0159" H 5100 6800 50  0001 C CNN
+F 0 "#PWR089" H 5100 6800 50  0001 C CNN
 F 1 "GND" H 5105 6877 50  0000 C CNN
 F 2 "" H 5100 7050 50  0001 C CNN
@@
 	4600 6750 4600 6650
 $Comp
-L power:GND #PWR0160
+L power:GND #PWR088
 U 1 1 63130F3E
 P 4600 7250
-F 0 "#PWR0160" H 4600 7000 50  0001 C CNN
+F 0 "#PWR088" H 4600 7000 50  0001 C CNN
 F 1 "GND" H 4605 7077 50  0000 C CNN
 F 2 "" H 4600 7250 50  0001 C CNN
@@
 	2750 5050 2750 5700
 $Comp
-L Device:R_Small_US R21
+L Device:R_Small_US R28
 U 1 1 6313BFA4
 P 2550 5700
-F 0 "R21" V 2345 5700 50  0000 C CNN
+F 0 "R28" V 2345 5700 50  0000 C CNN
 F 1 "NP" V 2436 5700 50  0000 C CNN
 F 2 "Resistor_SMD:R_0402_1005Metric" H 2550 5700 50  0001 C CNN
@@
 Text Notes 4350 4750 2    98   ~ 0
 Gyroscopic/Acceleration Sensor
-Text HLabel 1650 1650 0    50   Input ~ 0
+Text HLabel 4600 950  2    50   Input ~ 0
+SENSOR_I2C_SCL
+Text HLabel 4600 1050 2    50   Input ~ 0
+SENSOR_I2C_SDA
+Text Label 4600 950  2    50   ~ 0
+SCL
+Text Label 4600 1050 2    50   ~ 0
 SDA
+Text Label 1650 1650 2    50   ~ 0
+SDA
+Text Label 2150 1750 0    50   ~ 0
+SCL
+Text Label 3200 6050 2    50   ~ 0
+SDA
+Text Label 3200 6250 2    50   ~ 0
+SCL
 $EndSCHEMATC
